File: Schematic/SamyKam.kicad_pcb (KiCad board)
At the start: 2 copper layers, 65 x 30 mm, 19 parts, among them IC1 ATTINY85-P, P1 OLED, U1 TC4424, U2 RPi_Hat

Commit message: Fix Connection Grounds
Parts:
- S1: value Control -> PEC11R-4215F-S0024
- U2: value RPi_Hat -> RPi_A+_B+_2B_Hat
Connections:
- P1 pad 4: GNDA -> GND
- S1 pad C: GNDA -> GND
- U2 pad 30: GNDA -> GND
- U2 pad 34: GNDA -> GND
- U2 pad 6: GNDA -> GND
Routing:
- net GND: track 29.5 -> 94.6 mm, vias 2 -> 1
- net GNDA: track 52.4 -> 0.00 mm
- added copper zone on B.Cu, net GND
- removed copper zone on B.Cu, net GNDA
